File: kicad/digital-control.sch (KiCad schematic (older format))
At the start: 37 parts, among them J1 SWD, J4 USB_OTG, U1 STM32F042KxT, U2 USBLC6-2

Commit message: Upgraded schematic to Kicad 5
Parts:
- C1, C10, C11, C12, C13, C2, C22, C23, C3, C4, C5, C6, C7, C8, C9: symbol C -> Device:C
- J1: symbol Conn_01x04 -> Connector_Generic:Conn_01x04
- J4: symbol USB_OTG -> Connector:USB_OTG
- L1: symbol L -> Device:L
- R1, R10, R11, R12, R13, R2, R24, R25, R26, R27, R3, R4, R5, R6, R7, R8, R9: symbol R -> Device:R
- U1: symbol STM32F042KxT -> midi-fader:STM32F042KxT
- U2: symbol USBLC6-2 -> midi-fader:USBLC6-2
