File: kicad/input.sch (KiCad schematic (older format))
At the start: 32 parts, among them J2 EXTERNAL_OUT, J3 EXTERNAL_IN, SW1 TR2-21-L5, SW2 TR2-21-L5, U6 74HC165, U7 STP08DP05

Commit message: Upgraded schematic to Kicad 5
Parts:
- C24, C25, C26: symbol C -> Device:C
- J2, J3: symbol Conn_02x08_Odd_Even -> Connector_Generic:Conn_02x08_Odd_Even
- R28, R29, R30, R31, R32, R33, R34, R35, R36, R37, R38, R39, R40, R41, R42, R43, R44, R45, R46, R47, R48: symbol R -> Device:R
- RV1, RV2: symbol POT -> Device:R_POT
- SW1, SW2: symbol SW_Push_LED -> Switch:SW_Push_LED
- U6: symbol 74HC165 -> midi-fader:74HC165
- U7: symbol STP08DP05 -> midi-fader:STP08DP05
Connections:
- wire segments 147 -> 167
