File: kicad/power-supplies.sch (KiCad schematic (older format))
At the start: 22 parts, among them U3 MCP1603, U4 MIC2776L, U5 MIC5501-XYM5

Commit message: Upgraded schematic to Kicad 5
Parts:
- C14, C15, C16, C17, C18, C19, C20, C21: symbol C -> Device:C
- L2: symbol L -> Device:L
- R14, R15, R16, R17, R18, R19, R20, R21, R22, R23: symbol R -> Device:R
- U3: symbol MCP1603 -> midi-fader:MCP1603
- U4: symbol MIC2776L -> midi-fader:MIC2776L
- U5: symbol MIC5501-XYM5 -> midi-fader:MIC5501-XYM5
Changed lines of the file:
@@
-EESchema Schematic File Version 2
-LIBS:power
-LIBS:device
-LIBS:switches
-LIBS:relays
-LIBS:motors
-LIBS:transistors
-LIBS:conn
-LIBS:linear
-LIBS:regul
-LIBS:74xx
-LIBS:cmos4000
-LIBS:adc-dac
-LIBS:memory
-LIBS:xilinx
-LIBS:microcontrollers
-LIBS:dsp
-LIBS:microchip
-LIBS:analog_switches
-LIBS:motorola
-LIBS:texas
-LIBS:intel
-LIBS:audio
-LIBS:interface
-LIBS:digital-audio
-LIBS:philips
-LIBS:display
-LIBS:cypress
-LIBS:siliconi
-LIBS:opto
-LIBS:atmel
-LIBS:contrib
-LIBS:valves
-LIBS:midi-fader
+EESchema Schematic File Version 4
 LIBS:midi-fader-cache
-EELAYER 25 0
+EELAYER 26 0
 EELAYER END
 $Descr A4 11693 8268
@@
 $EndDescr
 $Comp
-L MCP1603 U3
+L midi-fader:MCP1603 U3
 U 1 1 5B3C69DA
 P 7300 2300
@@
 $EndComp
 $Comp
-L MIC5501-XYM5 U5
+L midi-fader:MIC5501-XYM5 U5
 U 1 1 5B3C6A50
 P 2900 3900
@@
 $EndComp
 $Comp
-L L L2
+L Device:L L2
 U 1 1 5B3CF824
 P 8150 2200
@@
 $EndComp
 $Comp
-L C C18
+L Device:C C18
 U 1 1 5B3CF8EC
 P 8950 2650
@@
 $EndComp
 $Comp
-L VBUS #PWR011
+L power:VBUS #PWR011
 U 1 1 5B3CF911
 P 1000 2100
@@
 $EndComp
 $Comp
-L C C14
+L Device:C C14
 U 1 1 5B3CF945
 P 1000 2450
@@
 $EndComp
 $Comp
-L C C15
+L Device:C C15
 U 1 1 5B3CF984
 P 1300 2450
@@
 $EndComp
 $Comp
-L R R15
+L Device:R R15
 U 1 1 5B3CF9F9
 P 2900 2450
@@
 $EndComp
 $Comp
-L R R18
+L Device:R R18
 U 1 1 5B3CFA6C
 P 2900 2950
@@
 $EndComp
 $Comp
-L R R20
+L Device:R R20
 U 1 1 5B3CFA99
 P 1900 3750
@@
 $EndComp
 $Comp
-L R R22
+L Device:R R22
 U 1 1 5B3CFAD8
 P 1900 4250
@@
 $EndComp
 $Comp
-L GND #PWR012
+L power:GND #PWR012
 U 1 1 5B3CFC0A
 P 1900 4600
@@
 $EndComp
 $Comp
-L R R14
+L Device:R R14
 U 1 1 5B3CFC3E
 P 1600 2450
@@
 $EndComp
 $Comp
-L R R17
+L Device:R R17
 U 1 1 5B3CFCD7
 P 9300 2650
@@
 VDD
 $Comp
-L MIC2776L U4
+L midi-fader:MIC2776L U4
 U 1 1 5B3D06F8
 P 5500 2800
@@
 $EndComp
 $Comp
-L GND #PWR013
+L power:GND #PWR013
 U 1 1 5B3D0BA6
 P 1000 2800
@@
 $EndComp
 $Comp
-L C C20
+L Device:C C20
 U 1 1 5B3D0D98
 P 3550 4150
@@
 $EndComp
 $Comp
-L C C21
+L Device:C C21
 U 1 1 5B3D0DE7
 P 3800 4150
@@
 $EndComp
 $Comp
-L C C19
+L Device:C C19
 U 1 1 5B3D1400
 P 4500 2900
@@
 $EndComp
 $Comp
-L GND #PWR014
+L power:GND #PWR014
 U 1 1 5B3D1467
 P 4500 3150
@@
 $EndComp
 $Comp
-L R R21
+L Device:R R21
 U 1 1 5B3D1C03
 P 4500 4050
@@
 $EndComp
 $Comp
-L R R23
+L Device:R R23
 U 1 1 5B3D1C09
 P 4500 4550
@@
 $EndComp
 $Comp
-L VDDA #PWR015
+L power:VDDA #PWR015
 U 1 1 5B3D1EBD
 P 3900 3700
@@
 $EndComp
 $Comp
-L GND #PWR016
+L power:GND #PWR016
 U 1 1 5B3D212E
 P 4500 4800
@@
 $EndComp
 $Comp
-L GND #PWR017
+L power:GND #PWR017
 U 1 1 5B3D21E1
 P 2900 3200
@@
 $EndComp
 $Comp
-L GND #PWR018
+L power:GND #PWR018
 U 1 1 5B3D2387
 P 5500 3200
@@
 $EndComp
 $Comp
-L C C16
+L Device:C C16
 U 1 1 5B3D2824
 P 8450 2650
@@
 $EndComp
 $Comp
-L C C17
+L Device:C C17
 U 1 1 5B3D286F
 P 8700 2650
@@
 15mA\n50mW\nRC=1.47ms
 $Comp
-L GND #PWR019
+L power:GND #PWR019
 U 1 1 5B3D2E2E
 P 8450 3000
@@
 $EndComp
 $Comp
-L R R16
+L Device:R R16
 U 1 1 5B3D350D
 P 6400 2450
@@
 $EndComp
 $Comp
-L R R19
+L Device:R R19
 U 1 1 5B3D35A4
 P 6400 3050
@@
 $EndComp
 $Comp
-L GND #PWR020
+L power:GND #PWR020
 U 1 1 5B3D365C
 P 6400 3300
@@
 $EndComp
 $Comp
-L VDD #PWR021
+L power:VDD #PWR021
 U 1 1 5B3D3EA7
 P 9300 2100
@@
 	1900 4400 1900 4600
 $Comp
-L GND #PWR022
+L power:GND #PWR022
 U 1 1 5B3D4CA8
 P 7300 2800
@@
 Vth=4.3V
 $Comp
-L VDDA #PWR023
+L power:VDDA #PWR023
 U 1 1 5B3D5A35
 P 4500 2600
@@
 VDDA_EN
 $Comp
-L PWR_FLAG #FLG024
+L power:PWR_FLAG #FLG024
 U 1 1 5B41D3F3
 P 8800 2100
